Commit message: fix(arm): merge per-link URDF collision meshes so full geometry survives
rdk's URDF parser keeps only the first <collision> element per link
(referenceframe/model_urdf.go falls back to Collision[0] after a capsule
check). The upstream SO-ARM100 links are multi-part assemblies, so passing
them as-is left each arm link with a single offset sub-part mesh -- collision
geometry that was both incomplete (rendered as sparse fragments) and visibly
misaligned within the link (18-54mm off the link's bulk).

Give each of the 5 arm links ONE merged collision mesh: arm/gen_collision_meshes.py
bakes every sub-part's <collision> origin into its vertices, concatenates them
per link, decimates to ~2500 tris, and writes arm/meshes/<link>_collision.stl.
arm/so101.urdf now references one mesh per link with an identity origin, so
rdk's Collision[0] is the full link. Kinematics/TCP unchanged (frame alignment
still 0.000mm/0.000rad).

New guard TestURDFCollisionCoversWholeLink asserts each URDF-mode link's
collision extent matches the JSON primitive (a lone sub-part can't), which
goes red on the old assets and green on the merged ones.

Replaces arm/gen_decimated_meshes.py + the 12 sub-part meshes.

Co-Authored-By: Claude Opus 4.8 (1M context) <noreply@anthropic.com>
Claude-Session: https://claude.ai/code/session_01Av6iEBnda6qM3Pg1C5cCZC

File: arm/so101.urdf (robot description, URDF)
Before this commit: robot so101_new_calib, 7 links, 6 joints
Links:
- link base_link: geometry collision mesh filename=meshes/base_link_collision.stl; visual mesh filename=meshes/base_link_collision.stl
- link gripper_link: geometry 
- link lower_arm_link: geometry collision mesh filename=meshes/lower_arm_link_collision.stl; visual mesh filename=meshes/lower_arm_link_collision.stl
- link shoulder_link: geometry collision mesh filename=meshes/shoulder_link_collision.stl; visual mesh filename=meshes/shoulder_link_collision.stl
- link upper_arm_link: geometry collision mesh filename=meshes/upper_arm_link_collision.stl; visual mesh filename=meshes/upper_arm_link_collision.stl
- link wrist_link: geometry collision mesh filename=meshes/wrist_link_collision.stl; visual mesh filename=meshes/wrist_link_collision.stl

Commit message: perf(arm): bake tool frame + names into so101.urdf for a smaller payload
Instead of grafting the tool frame and renaming frames in memory (which forced
re-serializing the whole model to SVA JSON so the edits would survive the
module gRPC boundary, ~5.9 MB with meshes embedded as base64), author
arm/so101.urdf so its raw form is already correct: links/joints use so101.json's
names (base..wrist, joints 1-5) and the chain ends at a "tool" leaf at
so101.json's TCP (joint-5 output + 180deg flip, via a tool_mount + fixed
tool_joint pair, since a revolute joint's child cannot carry the extra
rotation). makeSO101ModelURDF now just parses the URDF, so it transmits AS URDF
with meshes sent separately as binary -- ~4.4 MB vs ~5.9 MB.

visualize_ee_frame still needs an in-memory placeholder box on the tool link
(baking it statically would add a spurious collision volume for everyone), so
that one path re-serializes to SVA JSON to carry the box across the wire; the
larger payload is incurred only when the marker is enabled.

Removes the now-dead graft/rename helpers (urdfGraftedOutIDs,
urdfToJSONFrameNames, so101JSONToolLink, urdfWristRollJointID). All URDF guards
still green, including TestURDFModelSurvivesSerialization (now exercising the
URDF-format round-trip).

Co-Authored-By: Claude Opus 4.8 (1M context) <noreply@anthropic.com>
Claude-Session: https://claude.ai/code/session_01Av6iEBnda6qM3Pg1C5cCZC

File: arm/so101.urdf (robot description, URDF)
Before this commit: robot so101_new_calib, 7 links, 6 joints
Links:
- removed link base_link
- removed link gripper_frame_link
- removed link gripper_link
- removed link lower_arm_link
- removed link shoulder_link
- removed link upper_arm_link
- removed link wrist_link
- added link base, mass 0.147; collision mesh filename=meshes/base_link_collision.stl; visual mesh filename=meshes/base_link_collision.stl
- added link lower_arm, mass 0.104; collision mesh filename=meshes/lower_arm_link_collision.stl; visual mesh filename=meshes/lower_arm_link_collision.stl
- added link shoulder, mass 0.100006; collision mesh filename=meshes/shoulder_link_collision.stl; visual mesh filename=meshes/shoulder_link_collision.stl
- added link tool
- added link tool_mount
- added link upper_arm, mass 0.103; collision mesh filename=meshes/upper_arm_link_collision.stl; visual mesh filename=meshes/upper_arm_link_collision.stl
- added link wrist, mass 0.079; collision mesh filename=meshes/wrist_link_collision.stl; visual mesh filename=meshes/wrist_link_collision.stl
Joints:
- removed joint elbow_flex
- removed joint gripper_frame_joint
- removed joint shoulder_lift
- removed joint shoulder_pan
- removed joint wrist_flex
- removed joint wrist_roll
- added joint 1: type revolute, parent base, child shoulder, origin xyz=0.0388353 -8.97657e-09 0.0624 rpy=3.14159 4.18253e-17 -3.14159, axis 0 0 1, limit lower=-1.91986 upper=1.91986 effort=10 velocity=10
- added joint 2: type revolute, parent shoulder, child upper_arm, origin xyz=-0.0303992 -0.0182778 -0.0542 rpy=-1.5708 -1.5708 0, axis 0 0 1, limit lower=-1.74533 upper=1.74533 effort=10 velocity=10
- added joint 3: type revolute, parent upper_arm, child lower_arm, origin xyz=-0.11257 -0.028 1.73763e-16 rpy=-3.63608e-16 8.74301e-16 1.5708, axis 0 0 1, limit lower=-1.69 upper=1.69 effort=10 velocity=10
- added joint 4: type revolute, parent lower_arm, child wrist, origin xyz=-0.1349 0.0052 3.62355e-17 rpy=4.02456e-15 8.67362e-16 -1.5708, axis 0 0 1, limit lower=-1.65806 upper=1.65806 effort=10 velocity=10
- added joint 5: type revolute, parent wrist, child tool_mount, origin xyz=5.55112e-17 -0.0611 0.0181 rpy=1.5708 0.0486795 3.14159, axis 0 0 1, limit lower=-2.74385 upper=2.84121 effort=10 velocity=10
- added joint tool_joint: type fixed, parent tool_mount, child tool, origin xyz=0 0 0 rpy=0 3.14159 0.0486795
